Commit message: Updated camera static transf pose

File: realsense2_camera/urdf/realsense_standalong_physical.urdf.xacro (robot description, xacro)
@@ -4,5 +4,5 @@
   <link name="root" />
   <xacro:sensor_d435 name="camera" topics_ns="camera" parent="root" publish_pointcloud="true">
-    <origin xyz="0 1.1 1.58" rpy="0 0.51 -1.57075" />
+    <origin xyz="1.5 0.0 0.96" rpy="0.0 0.0 3.141592" />
   </xacro:sensor_d435>
   <gazebo>

Commit message: All Changes

File: realsense2_camera/urdf/realsense_standalong_physical.urdf.xacro (robot description, xacro)
@@ -4,5 +4,5 @@
   <link name="root" />
   <xacro:sensor_d435 name="camera" topics_ns="camera" parent="root" publish_pointcloud="true">
-    <origin xyz="1.5 0.0 0.96" rpy="0.0 0.0 3.141592" />
+    <origin xyz="-0.2 -0.35 1.23" rpy="0.09 0.28 1.5" />
   </xacro:sensor_d435>
   <gazebo>

File: realsense2_description/urdf/_d435.urdf.xacro (robot description, xacro)
@@ -57,4 +57,6 @@
         <geometry>
         <box size="${d435_cam_depth} ${d435_cam_width} ${d435_cam_height}"/>
+        <!-- <mesh filename="package://realsense2_description/meshes/d435.dae" /> -->
+        <!--<box size="0.03 0.1 0.035 "/> -->
         </geometry>
       </collision>

File: realsense2_description/urdf/test_d435_camera.urdf.xacro (robot description, xacro)
@@ -4,5 +4,5 @@
   <link name="root" />
   <xacro:sensor_d435 name="camera" topics_ns="camera" parent="root" publish_pointcloud="true">
-    <origin xyz="2.2 0 1.6" rpy="0 0.349066 3.1415" />
+    <origin xyz="0 -0.35 1.4" rpy="0 0.7853982 1.570796" />
   </xacro:sensor_d435>
   <gazebo>

Commit message: Slight changes in camera coordinates

File: realsense2_camera/urdf/realsense_standalong_physical.urdf.xacro (robot description, xacro)
@@ -4,5 +4,5 @@
   <link name="root" />
   <xacro:sensor_d435 name="camera" topics_ns="camera" parent="root" publish_pointcloud="true">
-    <origin xyz="-0.2 -0.35 1.23" rpy="0.09 0.28 1.5" />
+    <origin xyz="-0.2 -0.335 1.23" rpy="0.09 0.28 1.55" />
   </xacro:sensor_d435>
   <gazebo>
